Commit message: Update robot.xacro

File: robot_description_pkg/urdf/robot.xacro (robot description, xacro)
@@ -36,5 +36,5 @@
         <child link="chassis"/>
   </joint>
-  <!-- FRONT RIGHT WHEEL LINK   -->
+  <!-- FRONT LEFT WHEEL LINK   -->
   <link name="front_left_wheel">
     <inertial>
@@ -46,5 +46,5 @@
       <origin rpy="0 1.5707 1.5707" xyz="0 0 0" />
       <geometry>
-        <cylinder length="0.04" radius="0.1"/>
+        <cylinder length="0.05" radius="0.1"/>
       </geometry>
     </collision>
@@ -63,5 +63,5 @@
     <axis rpy="0 0 0" xyz="0 1 0"/>
   </joint>
-  <!-- BACk RIGHT WHEEL LINK    -->
+  <!-- BACk LEFT WHEEL LINK    -->
   <link name="back_left_wheel">
     <inertial>
@@ -73,5 +73,5 @@
       <origin rpy="0 1.5707 1.5707" xyz="0 0 0" />
       <geometry>
-        <cylinder length="0.04" radius="0.1"/>
+        <cylinder length="0.05" radius="0.1"/>
       </geometry>
     </collision>
@@ -90,5 +90,5 @@
     <axis rpy="0 0 0" xyz="0 1 0"/>
   </joint>
-  <!-- FRONT LEFTT WHEEL LINK   -->
+  <!-- FRONT RIGHT WHEEL LINK   -->
   <link name="front_right_wheel">
     <inertial>
@@ -127,5 +127,5 @@
       <origin rpy="0 1.5707 1.5707" xyz="0 0 0" />
       <geometry>
-        <cylinder length="0.04" radius="0.1"/>
+        <cylinder length="0.05" radius="0.1"/>
       </geometry>
     </collision>

Commit message: Update robot.xacro

File: robot_description_pkg/urdf/robot.xacro (robot description, xacro)
@@ -5,10 +5,4 @@
  <link name="odom">
   </link>
-  <link name="base_link">
-  </link>
-   <joint name="joint_base" type="fixed">
-        <parent link="odom"/>
-        <child link="base_link"/>
-  </joint>
   <!-- CHASSIS LINK -->
   <link name="chassis">
@@ -33,5 +27,5 @@
   </link>
   <joint name="joint_chassis" type="fixed">
-        <parent link="base_link"/>
+        <parent link="odom"/>
         <child link="chassis"/>
   </joint>
